File: Can.sch (KiCad schematic (older format))
At the start: 52 parts, among them IC1 ATMEGA328P-A, K1 HK4100F, K2 HK4100F, P3 CONN_01X03, P4 CONN_01X03, P5 CONN_01X02, P6 CONN_01X02, Q1 BC808-40, Q2 BC808-40, SW1 SW_PUSH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

Commit message: fix
Parts:
- removed U2: MCP2515, Housings_SOIC:SOIC-18_7.5x11.6mm_Pitch1.27mm, symbol MCP2515
Changed lines of the file:
@@
 LIBS:w_transistor
 LIBS:w_vacuum
-LIBS:HK4100F
-LIBS:MCP2515 E
-LIBS:mylib
-LIBS:acs712
-LIBS:Can-cache
 EELAYER 25 0
 EELAYER END
@@
 $EndComp
 $Comp
-L MCP2515 U2
-U 1 1 578B8152
-P 6050 3200
-F 0 "U2" H 6050 3100 50  0000 C CNN
-F 1 "MCP2515" H 6050 3300 50  0000 C CNN
-F 2 "Housings_SOIC:SOIC-18_7.5x11.6mm_Pitch1.27mm" H 6050 3200 50  0001 C CNN
-F 3 "DOCUMENTATION" H 6050 3200 50  0001 C CNN
-	1    6050 3200
-	-1   0    0    1
-$EndComp
-$Comp
